File: pcb/33220a_001.kicad_pcb (KiCad board)
At the start: 2 copper layers, 40 x 51.5 mm, 54 parts, among them J1 Conn_Coaxial, J2 Conn_Coaxial, P1 Conn_01x10_Socket, T1 TC1-1TX+, T2 TC1-1TX+, U1 LM361M, U2 74AC14

Commit message: added pics and added units
Parts:
- C10, C4: value 10 -> 10u
Changed lines of the file:
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@@
 			)
 		)
-		(property "Value" "10"
+		(property "Value" "10u"
 			(at 0 -1.68 90)
 			(layer "B.Fab")
@@
 			)
 		)
-		(property "Value" "10"
+		(property "Value" "10u"
 			(at 0 -1.68 90)
 			(layer "B.Fab")
